File: schem/LED_driver/CH_5.sch (KiCad schematic (older format))
At the start: 166 parts, among them J36 Screw_Terminal_01x04, J37 Screw_Terminal_01x02, J38 Screw_Terminal_01x02, J39 Screw_Terminal_01x02, J40 Screw_Terminal_01x02, J41 Screw_Terminal_01x02, U38 LM3406, U39 LM3406, U40 LM3406, U41 LM3406, U42 LM3406

Commit message: Start Programm
Начало настройки проекта. добавил файлы modbus, настроил проект под C++
Parts:
- removed J36: Screw_Terminal_01x04, TerminalBlock:TerminalBlock_bornier-4_P5.08mm, symbol Connector:Screw_Terminal_01x04
- added J1: Screw_Terminal_01x02, TerminalBlock:TerminalBlock_bornier-2_P5.08mm, symbol Connector:Screw_Terminal_01x02
Connections:
- net labels added: BUS1
- wire segments 543 -> 474
