File: schem/LED_driver/LED_driver.sch (KiCad schematic (older format))
At the start: 922 parts, among them J1 Screw_Terminal_01x02, J10 Screw_Terminal_01x02, J11 Screw_Terminal_01x02, J12 Screw_Terminal_01x02, J13 Screw_Terminal_01x02, J14 Screw_Terminal_01x02, J15 Screw_Terminal_01x02, J16 Screw_Terminal_01x02, J17 Screw_Terminal_01x02, J18 Screw_Terminal_01x02, J19 Screw_Terminal_01x02, J2 Screw_Terminal_01x02, J20 Screw_Terminal_01x02, J21 Screw_Terminal_01x02, J22 Screw_Terminal_01x02, J23 Screw_Terminal_01x02, J24 Screw_Terminal_01x02, J25 Screw_Terminal_01x02, J26 Screw_Terminal_01x02, J27 Screw_Terminal_01x02, J28 Screw_Terminal_01x02, J29 Screw_Terminal_01x02, J3 Screw_Terminal_01x02, J30 Screw_Terminal_01x02, J31 SWD, J32 RJ45_Shielded, J33 RJ45_Shielded, J34 DEBUG, J35 Screw_Terminal_01x02, J4 Screw_Terminal_01x02, J5 Screw_Terminal_01x02, J6 Screw_Terminal_01x02, J7 Screw_Terminal_01x02, J8 Screw_Terminal_01x02, J9 Screw_Terminal_01x02, SW1 SW_DIP_x01, U1 LM3406, U10 LM3406, U11 LM3406, U12 LM3406, U13 LM3406, U14 LM3406, U15 LM3406, U16 LM3406, U17 LM3406, U18 LM3406, U19 LM3406, U2 LM3406, U20 LM3406, U21 LM3406, U22 LM3406, U23 LM3406, U24 LM3406, U25 LM3406, U26 74HC595, U27 74HC595, U28 TL431LP, U29 STM32F303VCTx, U3 LM3406, U30 MCP2551-I_SN, U31 LM1117-3.3, U32 74HC595, U33 GD25Q16C, U34 MAX3485, U35 ISO7341C, U36 LM2596S-ADJ, U37 74HC595, U4 LM3406, U5 LM3406, U6 LM3406, U7 LM3406, U8 LM3406, U9 LM3406, Y1 Crystal_Small

Commit message: Start Programm
Начало настройки проекта. добавил файлы modbus, настроил проект под C++
Parts:
- removed C1, C10, C101, C103, C11, C111, C113, C121, C122, C127, C128, C130, C131, C141, C143, C151, C153, C161, C162, C167, C168, C170, C171, C181, C183, C191, C193, C2, C21, C23, C31, C33, C41, C42, C47, C48, C50, C51, C61, C63, C7, C71, C73, C8, C81, C82, C87, C88, C90, C91: 0.1mkF, Capacitor_SMD:C_0805_2012Metric, symbol Device:C
- removed C102, C104, C126, C129, C142, C144, C166, C169, C182, C184, C22, C24, C46, C49, C6, C62, C64, C86, C89, C9: 470mkF, Capacitor_THT:CP_Radial_D10.0mm_P5.00mm, symbol Device:CP
- removed C112, C114, C152, C154, C192, C194, C32, C34, C72, C74: 1mkF, Capacitor_SMD:C_0805_2012Metric, symbol Device:C
- removed D1, D2, D21, D22, D26, D27, D41, D42, D46, D47, D6, D61, D62, D66, D67, D7, D81, D82, D86, D87: D_Schottky, Diode_SMD:D_SMC, symbol Device:D_Schottky
- removed D11, D12, D31, D32, D51, D52, D71, D72, D91, D92: Si2300, Package_TO_SOT_SMD:SOT-23, symbol Transistor_FET:Si2300
- removed D16, D17, D36, D37, D56, D57, D76, D77, D96, D97: lmc7101, Package_TO_SOT_SMD:SOT-23-5, symbol Amplifier_Operational:lmc7101
- removed J1, J11, J12, J16, J17, J2, J21, J22, J26, J27, J6, J7: Screw_Terminal_01x02, TerminalBlock:TerminalBlock_bornier-2_P5.08mm, symbol Connector:Screw_Terminal_01x02
- removed L1, L11, L12, L16, L17, L2, L21, L22, L6, L7: 22mkH, Inductor_SMD:L_10.4x10.4_H4.8, symbol Device:L_Small
- removed R1, R101, R102, R11, R12, R166, R167, R171, R172, R181, R182, R191, R192, R2, R256, R257, R261, R262, R271, R272, R281, R282, R346, R347, R351, R352, R361, R362, R371, R372, R436, R437, R441, R442, R76, R77, R81, R82, R91, R92: 1K, Resistor_SMD:R_0805_2012Metric, symbol Device:R
- removed R106, R117, R16, R196, R207, R27, R286, R297, R376, R387: 100, Resistor_SMD:R_0805_2012Metric, symbol Device:R
- removed R107, R108, R109, R110, R111, R112, R113, R114, R115, R116, R118, R119, R120, R121, R122, R123, R124, R125, R126, R127, R17, R18, R19, R197, R198, R199, R20, R200, R201, R202, R203, R204, R205, R206, R208, R209, R21, R210, R211, R212, R213, R214, R215, R216, R217, R22, R23, R24, R25, R26, R28, R287, R288, R289, R29, R290, R291, R292, R293, R294, R295, R296, R298, R299, R30, R300, R301, R302, R303, R304, R305, R306, R307, R31, R32, R33, R34, R35, R36, R37, R377, R378, R379, R380, R381, R382, R383, R384, R385, R386, R388, R389, R390, R391, R392, R393, R394, R395, R396, R397: 1R, Resistor_SMD:R_1206_3216Metric, symbol Device:R
- removed R161, R162, R186, R187, R251, R252, R276, R277, R341, R342, R366, R367, R431, R432, R6, R7, R71, R72, R96, R97: 100K, Resistor_SMD:R_0805_2012Metric, symbol Device:R
- removed R176, R177, R266, R267, R356, R357, R446, R447, R86, R87: 10K, Resistor_SMD:R_0805_2012Metric, symbol Device:R
- removed U1, U11, U12, U16, U17, U2, U21, U22, U6, U7: LM3406, Package_SO:TSSOP-14-1EP_4.4x5mm_P0.65mm, symbol LED_driver-rescue:LM3406-Regulator_Switching
